File: project/LazuriteBLE/LazuriteBLE_rev1.brd (EAGLE design)
At the start: 32 x 24 mm, 21 parts

Commit message: update Lazurite BLE
Parts:
- added C16: 22u, rcl:C1206
- moved C14 4.96 mm to (6.99, 7.62), turned to 90 degrees
- moved U$6 1.93 mm to (11.4, 6.67), turned to 180 degrees
- moved C8 1.00 mm to (13.3, 6.67), turned to 270 degrees
Connections:
- net +5V: now also C16.1
- net BLE_CTS: now also U$1.37; no longer U$1.20
- net BLE_RX: now also U$1.19; no longer U$1.37
- net BLE_TX: now also U$1.20; no longer U$1.38
- net BLE_WAKEUP: now also U$1.38; no longer U$1.19
- net GND: now also C16.2
Routing:
- net GND: track 16.5 -> 40.7 mm, vias 8 -> 13
- net BLE_WAKEUP: track 23.8 -> 6.11 mm, vias 3 -> 1
- net BLE_RX: track 12.3 -> 29.5 mm, vias 2 -> 3
- net BLE_CTS: track 17.4 -> 4.94 mm, vias 4 -> 1
- net BLE_TX: track 15.8 -> 25.5 mm, vias 2 -> 3
- net +3V3: track 22.0 -> 27.3 mm, vias 9 -> 6
- net P50: track 15.3 -> 11.5 mm, vias 3 -> 1
- net P30: track 8.27 -> 6.12 mm, vias 1 -> 0
- net P31: track 10.0 -> 8.16 mm, vias 1 -> 0
- net +5V: track 13.6 -> 11.9 mm, vias 2 -> 0
- net N$1: track 7.25 -> 8.20 mm
- net P33: track 20.3 -> 21.2 mm, vias 2 -> 3
- net N$3: track 8.20 -> 8.76 mm
- net P23: track 13.6 -> 13.4 mm, vias 3 -> 2
- net P34: vias 2 -> 1
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- added copper zone on layer 3, net +3V3
- added copper zone on layer 2, net GND
- removed copper zone on layer 16, net +3V3
- removed copper zone on layer 1, net GND
