File: project/LazuriteBLE/LazuriteBLE_rev1_1.brd (EAGLE design)
At the start: 32 x 24 mm, 22 parts

Commit message: modify lazurite ble  - add reset button.
Parts:
- added SW1: SKSGACE010, lz-shield:SKSGACE010
Connections:
- net GND: now also SW1.2, SW1.4, SW1.5, SW1.6
- net RESETN: now also SW1.1, SW1.3
Routing:
- net RESETN: track 0.00 -> 11.3 mm, vias 0 -> 1
- net GND: track 40.7 -> 47.1 mm, vias 13 -> 14
Changed lines of the file:
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@@
 <layer number="21" name="tPlace" color="7" fill="1" visible="yes" active="yes"/>
 <layer number="22" name="bPlace" color="7" fill="1" visible="yes" active="yes"/>
-<layer number="23" name="tOrigins" color="15" fill="1" visible="no" active="yes"/>
+<layer number="23" name="tOrigins" color="15" fill="1" visible="yes" active="yes"/>
 <layer number="24" name="bOrigins" color="15" fill="1" visible="yes" active="yes"/>
 <layer number="25" name="tNames" color="7" fill="1" visible="no" active="yes"/>
@@
 <layer number="49" name="Reference" color="7" fill="1" visible="yes" active="yes"/>
 <layer number="50" name="dxf" color="7" fill="1" visible="no" active="no"/>
-<layer number="51" name="tDocu" color="7" fill="1" visible="no" active="yes"/>
+<layer number="51" name="tDocu" color="7" fill="1" visible="yes" active="yes"/>
 <layer number="52" name="bDocu" color="7" fill="1" visible="yes" active="yes"/>
 <layer number="53" name="tGND_GNDA" color="7" fill="9" visible="no" active="no"/>
@@
 <attribute name="VALUE" x="11.43" y="5.3975" size="1.27" layer="27" rot="R90"/>
 </element>
+<element name="SW1" library="lz-shield" package="SKSGACE010" value="SKSGACE010" x="2.8575" y="15.5575"/>
 </elements>
 <signals>
@@
 <wire x1="22.925" y1="15.205" x2="22.925" y2="16.445" width="0.3048" layer="1"/>
 <wire x1="22.925" y1="16.445" x2="22.86" y2="16.51" width="0.3048" layer="1"/>
+<contactref element="SW1" pad="4"/>
+<via x="3.4925" y="15.5575" extent="1-16" drill="0.3048"/>
+<contactref element="SW1" pad="6"/>
+<contactref element="SW1" pad="2"/>
+<contactref element="SW1" pad="5"/>
+<wire x1="1.145" y1="15.5575" x2="3.4925" y2="15.5575" width="0.2032" layer="1"/>
+<wire x1="1.295" y1="14.145" x2="1.295" y2="15.4075" width="0.2032" layer="1"/>
+<wire x1="1.295" y1="15.4075" x2="1.145" y2="15.5575" width="0.2032" layer="1"/>
+<wire x1="3.4925" y1="15.5575" x2="4.57" y2="15.5575" width="0.2032" layer="1"/>
+<wire x1="4.57" y1="15.5575" x2="4.57" y2="14.295" width="0.2032" layer="1"/>
+<wire x1="4.57" y1="14.295" x2="4.42" y2="14.145" width="0.2032" layer="1"/>
 </signal>
 <signal name="P04">
@@
 <wire x1="12.3825" y1="16.1925" x2="6.0325" y2="16.1925" width="0.2032" layer="2"/>
 <via x="6.0325" y="16.1925" extent="1-16" drill="0.3048"/>
-<wire x1="6.795" y1="12.7" x2="6.0325" y2="12.7" width="0.2032" layer="1"/>
-<wire x1="6.0325" y1="12.7" x2="5.715" y2="13.0175" width="0.2032" layer="1"/>
-<wire x1="5.715" y1="13.0175" x2="5.715" y2="15.875" width="0.2032" layer="1"/>
+<wire x1="6.795" y1="12.7" x2="6.795" y2="14.16" width="0.2032" layer="1"/>
+<wire x1="6.795" y1="14.16" x2="6.35" y2="14.605" width="0.2032" layer="1"/>
+<wire x1="6.35" y1="14.605" x2="6.0325" y2="14.605" width="0.2032" layer="1"/>
+<wire x1="6.0325" y1="14.605" x2="5.715" y2="14.9225" width="0.2032" layer="1"/>
+<wire x1="5.715" y1="14.9225" x2="5.715" y2="15.875" width="0.2032" layer="1"/>
 <wire x1="5.715" y1="15.875" x2="6.0325" y2="16.1925" width="0.2032" layer="1"/>
 </signal>
@@
 <signal name="RESETN">
 <contactref element="U$1" pad="1"/>
+<contactref element="SW1" pad="3"/>
+<contactref element="SW1" pad="1"/>
+<wire x1="5.08" y1="16.51" x2="4.62" y2="16.97" width="0.2032" layer="1"/>
+<wire x1="4.62" y1="16.97" x2="4.42" y2="16.97" width="0.2032" layer="1"/>
+<wire x1="1.295" y1="16.97" x2="4.42" y2="16.97" width="0.2032" layer="1"/>
+<wire x1="8.575" y1="11.855" x2="6.56" y2="11.855" width="0.2032" layer="16"/>
+<wire x1="6.56" y1="11.855" x2="5.715" y2="12.7" width="0.2032" layer="16"/>
+<via x="5.715" y="12.7" extent="1-16" drill="0.3048"/>
+<wire x1="5.715" y1="12.7" x2="5.715" y2="13.97" width="0.2032" layer="1"/>
+<wire x1="5.715" y1="13.97" x2="5.08" y2="14.605" width="0.2032" layer="1"/>
+<wire x1="5.08" y1="14.605" x2="5.08" y2="16.51" width="0.2032" layer="1"/>
 </signal>
 <signal name="P30">

Commit message: update libraries: add 1pin mark update Lazurite BLE: add silk of LOGO, board name, and pin number of Lazurite BLE. create SPI_Sensor_Shield.
Parts:
- added U$2: (no value), lazurite:LOGO
Other:
- board text added: "0"
- board text added: "1"
- board text added: "13-4"
- board text added: "Lazurite BLE"
- board text added: "V,G,14-19,3,2"
- board text added: "developed in Japan made in Japan"
Changed lines of the file:
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@@
 <layer number="24" name="bOrigins" color="15" fill="1" visible="yes" active="yes"/>
 <layer number="25" name="tNames" color="7" fill="1" visible="no" active="yes"/>
-<layer number="26" name="bNames" color="7" fill="1" visible="yes" active="yes"/>
+<layer number="26" name="bNames" color="7" fill="1" visible="no" active="yes"/>
 <layer number="27" name="tValues" color="7" fill="1" visible="no" active="yes"/>
 <layer number="28" name="bValues" color="7" fill="1" visible="no" active="yes"/>
@@
 <layer number="47" name="Measures" color="7" fill="1" visible="no" active="yes"/>
 <layer number="48" name="Document" color="7" fill="1" visible="no" active="yes"/>
-<layer number="49" name="Reference" color="7" fill="1" visible="yes" active="yes"/>
+<layer number="49" name="Reference" color="7" fill="1" visible="no" active="yes"/>
 <layer number="50" name="dxf" color="7" fill="1" visible="no" active="no"/>
-<layer number="51" name="tDocu" color="7" fill="1" visible="yes" active="yes"/>
-<layer number="52" name="bDocu" color="7" fill="1" visible="yes" active="yes"/>
+<layer number="51" name="tDocu" color="7" fill="1" visible="no" active="yes"/>
+<layer number="52" name="bDocu" color="7" fill="1" visible="no" active="yes"/>
 <layer number="53" name="tGND_GNDA" color="7" fill="9" visible="no" active="no"/>
 <layer number="54" name="bGND_GNDA" color="1" fill="9" visible="no" active="no"/>
@@
 <text x="27.305" y="0.9525" size="1.27" layer="22" font="fixed" rot="SMR90">Lazurite BLE rev1</text>
 <text x="29.845" y="0.9525" size="1.778" layer="22" rot="MR90">LAPIS</text>
+<text x="19.685" y="1.5875" size="0.8128" layer="21" font="fixed">13-4</text>
+<text x="19.685" y="21.9075" size="0.8128" layer="21" font="fixed">V,G,14-19,3,2</text>
+<text x="9.8425" y="19.3675" size="1.4224" layer="21" font="fixed">Lazurite BLE</text>
+<text x="10.795" y="16.8275" size="0.8128" layer="21" font="fixed">developed in Japan
+made in Japan</text>
+<text x="0.9525" y="13.0175" size="0.8128" layer="21" font="fixed">1</text>
+<text x="3.175" y="13.0175" size="0.8128" layer="21" font="fixed">0</text>
 </plain>
 <attributes>
@@
 </element>
 <element name="SW1" library="lz-shield" package="SKSGACE010" value="SKSGACE010" x="2.8575" y="15.5575"/>
+<element name="U$2" library="lazurite" package="LOGO" value="" x="5.08" y="17.4625"/>
 </elements>
 <signals>
