File: project/LazuriteBLE/170217_LazuriteBLE/eagle/LazuriteBLE_rev1.brd (EAGLE design)
At the start: 32 x 24 mm, 22 parts

Commit message: update Lazurite BLE
Parts:
- removed R1: 100K, rcl:R0402
- added C16: 22u, rcl:C1206
- U1: device lazurite:LAZURITE920J_2 -> lazurite:LAZURITE920J2
- moved C2 16.0 mm to (6.35, 18.7), turned to 90 degrees
- moved C4 8.67 mm to (16.2, 8.57), flipped to the bottom, turned to 180 degrees
- moved C14 5.12 mm to (6.99, 7.62), turned to 90 degrees
- moved C8 2.93 mm to (13.3, 6.67), turned to 270 degrees
- moved U$6 2.56 mm to (11.4, 6.67)
- moved C3 1.00 mm to (16.2, 6.03), turned to 180 degrees
- moved C17 0.63 mm to (7.62, 4.45)
- moved C18 0.63 mm to (10.8, 4.45)
- moved C5 0.45 mm to (16.2, 7.30)
- turned R14 to 180 degrees
- turned R15 to 180 degrees
Connections:
- removed net N$16: R1.2, U$6.5
- net +5V: now also C16.1
- net BLE_CTS: now also U$1.37; no longer U$1.20
- net BLE_PRG: now also U$1.21; no longer U$1.19
- net BLE_RX: now also U$1.19; no longer U$1.37
- net BLE_TX: now also U$1.20; no longer U$1.38
- net BLE_WAKEUP: now also U$1.38; no longer U$1.21
- net GND: now also C16.2, U$6.5; no longer R1.1
Routing:
- net GND: track 3.07 -> 40.7 mm, vias 1 -> 13
- net BLE_RX: track 0.00 -> 29.5 mm, vias 0 -> 3
- net RF_RSTBI: track 0.00 -> 27.0 mm, vias 0 -> 3
- net BLE_TX: track 0.00 -> 25.5 mm, vias 0 -> 3
- net +3V3: track 4.99 -> 27.3 mm, vias 3 -> 6
- net P33: track 0.00 -> 21.2 mm, vias 0 -> 3
- net P45: track 0.00 -> 21.1 mm, vias 0 -> 1
- net P44: track 0.00 -> 20.2 mm, vias 0 -> 2
- net P32: track 0.00 -> 19.5 mm, vias 0 -> 2
- net P36: track 0.00 -> 17.9 mm, vias 0 -> 1
- net BLE_PRG: track 0.00 -> 16.9 mm, vias 0 -> 3
- net P37: track 0.00 -> 16.8 mm, vias 0 -> 1
- net P42: track 0.00 -> 16.5 mm, vias 0 -> 1
- net P51: track 0.00 -> 15.3 mm, vias 0 -> 2
- net P43: track 0.00 -> 15.3 mm, vias 0 -> 1
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- added copper zone on layer 3, net +3V3
- added copper zone on layer 2, net GND
Other:
- board text added: "LAPIS"
- board text added: "Lazurite BLE rev1"
