File: project/LazuriteBLE/170217_LazuriteBLE/eagle/LazuriteBLE_rev1.sch (EAGLE design)
At the start: 23 parts

Commit message: update Lazurite BLE
Parts:
- removed R1: 100K, rcl:R-US_R0402
- removed R3: 47k, rcl:R-US_R0402
- added C16: 22u, rcl:C-EUC1206
- U$6: value BHXXPB1WFV -> BH33PB1WFV
- U1: device lazurite:LAZURITE920JLAZURITE920J -> lazurite:LAZURITE920J
Connections:
- net RF_CSBI renamed RF_WAKEUP
- removed net 3V: C8.1, U$6.VOUT
- removed net 5V: C14.1, U$6.STBY, U$6.VIN
- removed net BLERSTB: U$4.7
- removed net CTS: U$4.16
- removed net IOREF: C1.1, C2.1, C5.1, R13.2, R14.1, R15.1, U$1.VDD1, U$1.VDD2, U$1.VREF
- removed net MISO0I: U$1.P01
- removed net MOSI0I: U$1.P00
- removed net N$10: U1B.TEST0
- removed net N$11: U1D.14
- removed net N$12: U1D.15
- removed net N$13: U1D.16
- removed net N$14: U1D.17
- removed net N$15: U1D.18
- removed net N$16: R1.2, U$6.SEL
- removed net N$17: U1D.19
- removed net N$18: U1D.3
- removed net N$20: U1D.2
- removed net N$21: U1C.4
- removed net N$23: U1C.5
- removed net N$24: U1C.6
- removed net N$25: U1C.7
- removed net N$26: U1C.8
- removed net N$27: U1C.9
- removed net N$28: U1C.10
- removed net N$29: U1C.11
- removed net N$30: U1C.12
- removed net N$31: U1C.13
- removed net N$6: U1B.1
- removed net N$8: U1B.TEST1N
- removed net N$9: U1B.0
- removed net NFC_IRQI: U$1.P55
- removed net PRG: U$4.13
- removed net RF_REGPDINI: U$1.P54
- removed net RTS: R3.2, U$4.19
- removed net RX: U$4.21
- removed net SCL0I: U$1.P41
- removed net SCLK0I: U$1.P02
- removed net TX: U$4.22
- new net BLE_CTS: U$1.P54, U$4.16
- new net BLE_GPIO0: U$1.P41, U$4.18
- new net BLE_PRG: U$1.P02, U$4.13
- new net BLE_RX: U$1.P00, U$4.21
- new net BLE_TX: U$1.P01, U$4.22
- new net BLE_WAKEUP: U$1.P55, U$4.19
- net +3V3: now also C1.1, C2.1, C5.1, C8.1, R13.2, R14.1, R15.1, U$1.VDD1, U$1.VDD2, U$1.VREF, U$6.VOUT
- net +5V: now also C14.1, C16.1, U$6.STBY, U$6.VIN
- net GND: now also C16.2, U$6.SEL; no longer R1.1, R3.1
- net P03: now also U1D.17
- net P20: now also U1D.14
- net P21: now also U1D.15
- net P22: now also U1D.16
- net P30: now also U1B.0
- net P31: now also U1B.1
- net P32: now also U1C.6
- net P33: now also U1C.7
- net P34: now also U1D.18
- net P35: now also U1D.19
- net P36: now also U1C.13
- net P37: now also U1C.10
- net P42: now also U1C.4
- net P43: now also U1C.5
- net P44: now also U1C.11
- net P45: now also U1C.12
- net P50: now also U1D.2
- net P52: now also U1C.9
- net P53: now also U1D.3
- net P57: now also U1C.8
- net RF_RSTBI: now also U$4.7
- net TEST0: now also U1B.TEST0
- net TEST1N: now also U1B.TEST1N
Other:
- note added: "RESET button追加"
