File: project/LazuriteRev3/lazurite_rev3_2.brd (EAGLE design)
At the start: 76.2 x 53.3 mm, 62 parts, among them IC1 FT232RQ

Commit message: update Lazurite BLE
Connections:
- net IOREF: now also R13.2
- net USBVDD: no longer R13.2
Routing:
- net IOREF: track 214.0 -> 230.4 mm, vias 18 -> 19
- net USBVDD: track 74.6 -> 66.0 mm, vias 6 -> 5
Changed lines of the file:
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@@
 <wire x1="66.167" y1="30.48" x2="66.04" y2="30.607" width="1.016" layer="2"/>
 <wire x1="66.04" y1="30.607" x2="66.04" y2="32.0675" width="1.016" layer="2"/>
+<contactref element="R13" pad="2"/>
+<wire x1="3.4775" y1="36.83" x2="3.4925" y2="36.83" width="0.2032" layer="1"/>
+<wire x1="3.4925" y1="36.83" x2="3.4925" y2="35.56" width="0.2032" layer="1"/>
+<via x="3.4925" y="35.56" extent="1-16" drill="0.3048"/>
+<wire x1="10.795" y1="32.385" x2="10.795" y2="29.845" width="0.2032" layer="3"/>
+<wire x1="10.795" y1="29.845" x2="12.065" y2="28.575" width="0.2032" layer="3"/>
+<wire x1="12.065" y1="28.575" x2="14.2875" y2="28.575" width="0.2032" layer="3"/>
+<wire x1="3.4925" y1="35.56" x2="7.62" y2="35.56" width="0.2032" layer="3"/>
+<wire x1="7.62" y1="35.56" x2="10.795" y2="32.385" width="0.2032" layer="3"/>
 </signal>
 <signal name="P20">
@@
 <contactref element="C20" pad="1"/>
 <contactref element="L1" pad="2"/>
-<contactref element="R13" pad="2"/>
 <wire x1="14.605" y1="17.16" x2="14.9225" y2="17.4775" width="0.3048" layer="1"/>
 <wire x1="14.9225" y1="17.4775" x2="14.9225" y2="18.7325" width="0.3048" layer="1"/>
@@
 <wire x1="14.59" y1="17.145" x2="14.605" y2="17.16" width="0.4064" layer="1"/>
 <wire x1="9.2075" y1="19.685" x2="10.4775" y2="20.955" width="1.016" layer="2"/>
-<wire x1="10.4775" y1="20.955" x2="10.4775" y2="38.1" width="1.016" layer="2"/>
-<wire x1="10.4775" y1="38.1" x2="10.4775" y2="42.545" width="1.016" layer="2"/>
+<wire x1="10.4775" y1="20.955" x2="10.4775" y2="42.545" width="1.016" layer="2"/>
 <wire x1="15.24" y1="46.355" x2="16.51" y2="46.355" width="1.016" layer="2"/>
-<wire x1="3.4775" y1="36.83" x2="3.4775" y2="38.085" width="0.4064" layer="1"/>
-<wire x1="3.4775" y1="38.085" x2="3.81" y2="38.4175" width="0.4064" layer="1"/>
-<wire x1="3.81" y1="38.4175" x2="10.16" y2="38.4175" width="0.4064" layer="2"/>
-<wire x1="10.16" y1="38.4175" x2="10.4775" y2="38.1" width="0.4064" layer="2"/>
 <wire x1="12.7" y1="43.83" x2="12.7" y2="46.0375" width="1.016" layer="1"/>
 <wire x1="14.605" y1="43.83" x2="12.7" y2="43.83" width="1.016" layer="1"/>
@@
 <wire x1="13.97" y1="46.355" x2="15.24" y2="46.355" width="1.016" layer="2"/>
 <wire x1="13.0175" y1="46.355" x2="16.51" y2="46.355" width="1.016" layer="1"/>
-<via x="3.81" y="38.4175" extent="1-16" drill="0.3048"/>
 <wire x1="12.08" y1="17.16" x2="14.605" y2="17.16" width="0.4064" layer="1"/>
 <via x="9.2075" y="16.8275" extent="1-16" drill="0.6096"/>
