File: project/LazuriteRev3/lazurite_rev3_2.sch (EAGLE design)
At the start: 60 parts, among them IC1 FT232RQ

Commit message: update Lazurite BLE
Connections:
- net IOREF: now also R13.2
- net USBVDD: no longer R13.2
Changed lines of the file:
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@@
 <wire x1="-185.42" y1="-2.54" x2="-185.42" y2="0" width="0.1524" layer="91"/>
+</segment>
+<segment>
+<pinref part="R13" gate="G$1" pin="2"/>
+<wire x1="-22.86" y1="104.14" x2="-22.86" y2="119.38" width="0.1524" layer="91"/>
+<label x="-22.86" y="119.38" size="1.778" layer="95"/>
 </segment>
 </net>
@@
 <junction x="-33.02" y="33.02"/>
 <wire x1="-33.02" y1="50.8" x2="-33.02" y2="114.3" width="0.1524" layer="91"/>
-<wire x1="-33.02" y1="114.3" x2="-22.86" y2="114.3" width="0.1524" layer="91"/>
-<wire x1="-22.86" y1="114.3" x2="-5.08" y2="114.3" width="0.1524" layer="91"/>
+<wire x1="-33.02" y1="114.3" x2="-5.08" y2="114.3" width="0.1524" layer="91"/>
 <wire x1="-5.08" y1="114.3" x2="7.62" y2="114.3" width="0.1524" layer="91"/>
 <wire x1="7.62" y1="114.3" x2="12.7" y2="114.3" width="0.1524" layer="91"/>
-<wire x1="-22.86" y1="114.3" x2="-22.86" y2="104.14" width="0.1524" layer="91"/>
-<pinref part="R13" gate="G$1" pin="2"/>
-<junction x="-22.86" y="114.3"/>
 <junction x="-5.08" y="114.3"/>
 <junction x="7.62" y="114.3"/>
 <pinref part="U$15" gate="G$1" pin="A"/>
-</segment>
-</net>
+<junction x="-33.02" y="50.8"/>
+</segment>
+</net>
