File: project/LazuriteRev3/lazurite_rev3_3.sch (EAGLE design)
At the start: 42 parts, among them IC1 FT232RQ

Commit message: fixed Pi Gateway2
Parts:
- removed C26: 0.1u, rcl:C-EUC0402
- removed JP2: (no value), pinhead:PINHD-2X20
- removed JP3: (no value), pinhead:PINHD-2X4
- removed R16, R17, R18, R19, R22: 10K, rcl:R-US_R0402
- removed R20: 0, rcl:R-US_R0402
- removed R21: NC, rcl:R-US_R0402
- added C10, C11, C12, C13, C7: 0.1u, rcl:C-EUC0402
- added C14: 0.01u, rcl:C-EUC0402
- added C15: 47u, rcl:C-EUC1210
- added C17, C18: 8p, rcl:C-EUC0402
- added C6: 10u, rcl:C-EUC0402
- added C8: 2.2u, rcl:C-EUC0402
- added R14, R15: 1K, rcl:R-US_R0402
- added R3: 10K, rcl:R-US_R0402
- added U$10: LAZURITE_BASIC, lazurite:LAZURITE_BASIC
- added U$12: XB-1-X, lz-shield:XB-1-X
- added U$13: PJ-102AH, lazurite:PJ-102AH
- added U$14, U$15: RB160MM, lazurite:RB160MM
- added U$17: SML-E12Y8W, lazurite:SML-E1X
- added U$18: SML-E13BC8T, lazurite:SML-E1X
- added U$20: DF40C-20DP-0.4V(51), lazurite:BP3596A
- added U$8: FXMA2102, lazurite:FXMA2102
- added U$9: FXMA108, lazurite:FXMA108
- R1: value 510 -> 100K
- R11, R12: value 1K -> 510
- R5, R6: value 510 -> 10K
- R9: value 10K -> NC
- U$2: value RT1A060AP -> TI-TS5A23159; device lz-shield:RT1A060AP -> lz-shield:TI-TS5A23159
- U$3: value TI-TS5A23159 -> NX3215SA; device lz-shield:TI-TS5A23159 -> lazurite:NX3215SA
- U$4: value DF40C-20DP-0.4V(51) -> MHS221; device lazurite:BP3596A -> lazurite:MHS221
- U$5: value SML-E13BC8T -> BA50BC0FP; device lazurite:SML-E1X -> lazurite:BA50BC0FP
- U$6: value SML-E12Y8W -> BHXXPB1WFV; device lazurite:SML-E1X -> lazurite:BHXXPB1WFV
Connections:
- removed net +3V3: JP2.1, JP2.17, R11.1, R12.1, R16.1, R17.1, R18.1, R19.1, R22.1, U$4.8, U$4.9
- removed net +5V: JP2.2, JP2.4, U$2.D1, U$2.D2, U$2.D3, U$2.D4, U$2.D6
- removed net +5V/1: C1.1, C16.1, C19.1, C2.1, C20.1, C24.1, C26.1, C5.1, IC1.VCC, IC1.VCCIO, JP3.1, R10.1, R13.2, R9.1, U$1.VDD1, U$1.VDD2, U$1.VREF, U$11G$2.1, U$2.S, U$3G$3.VDD
- removed net I2C_SCL: JP2.5, R17.2, U$4.1
- removed net I2C_SDA: JP2.3, R16.2, U$4.2
- removed net LED_RX: JP2.33, U$6.C
- removed net LED_TX: JP2.31, U$5.C
- removed net M2P: JP2.7
- removed net MISO: JP2.21, U$4.12
- removed net MOSI: JP2.19, U$4.16
- removed net N$10 (its old number): JP2.29
- removed net N$12: JP2.37
- removed net N$13: JP2.40
- removed net N$15: JP2.38
- removed net N$19 (its old number): IC1.CBUS1, R5.2
- removed net N$20: JP2.28
- removed net N$21: JP2.22
- removed net N$28: R1.1, U$2.G
- removed net N$29: JP2.18
- removed net N$30: JP2.16
- removed net N$34: JP2.10
- removed net N$36: U$4.GND2
- removed net N$37: R11.2, U$6.A
- removed net N$38: R12.2, U$5.A
- removed net N$4 (its old number): IC1.!RTS, U$3G$1.NO
- removed net P2M: JP2.8
- removed net RF_CSB0: JP2.24, R19.2, R20.2
- removed net RF_CSB1: JP2.26, R21.2, R22.2
- removed net SCLK: JP2.23, U$4.14
- new net 3V: C11.1, C13.1, C8.1, R5.2, R6.2, U$10.3V$1, U$20.8, U$20.9, U$4.1, U$4.4, U$6.VOUT, U$8.VCCB, U$9.VCCB
- new net 5V: C14.1, C16.1, C20.1, IC1.VCC, U$10.5V, U$15.C, U$4.3, U$4.6, U$5.OUT, U$6.STBY, U$6.VIN
- new net IOREF: C1.1, C10.1, C12.1, C19.1, C2.1, C24.1, C5.1, C6.1, C7.1, IC1.VCCIO, R13.2, R14.1, R15.1, R3.2, R4.2, R9.1, U$1.VDD1, U$1.VDD2, U$1.VREF, U$10.AREF, U$10.IOREF$1, U$10.IOREF$2, U$12.8_2, U$2G$3.VDD, U$4.2, U$4.5, U$8.OE, U$8.VCCA, U$9.VCCA
- new net MISO0: U$20.12, U$9.B2
- new net MISO0I: U$1.P01, U$9.A2
- new net MOSI0: U$20.16, U$9.B6
- new net MOSI0I: U$1.P00, U$9.A6
- new net N$22: R15.2, U$18.A
- new net N$24: U$20.GND2
- new net N$6: IC1.CBUS0, R12.2
- new net NFC_IRQI: U$1.P55
- new net RF_CSBI: U$1.P10, U$9.A5
- new net RF_IRQI: U$1.P47, U$9.A3
- new net RF_REGPDINI: U$1.P54, U$9.A1
- new net RF_RSTBI: U$1.P11, U$9.AO
- new net SCL0: R5.1, U$20.1, U$8.B0
- new net SCL0I: R4.1, U$1.P41, U$8.A0
- new net SCLK0: U$20.14, U$9.B4
- new net SCLK0I: U$1.P02, U$9.A4
- new net SDA0: R6.1, U$20.2, U$8.B1
- new net SDA0I: R3.1, U$1.P40, U$8.A1
- new net USBVDD: U$11G$2.1, U$15.A
- new net VIN: C15.1, U$10.VIN, U$14.C, U$5.VCC
- net AVDD_MON: now also U$20.7; no longer U$4.7
- net BOOT_WRITE: now also R10.1, R9.2, U$2G$1.IN, U$2G$2.IN; no longer R4.1, U$3G$1.IN, U$3G$2.IN
- net EEP_WP: now also U$20.18, U$9.B7; no longer U$4.18
- net GND: now also C10.2, C11.2, C12.2, C13.2, C14.2, C15.2, C17.2, C18.2, C6.2, C7.2, C8.2, R1.1, R10.2, U$10.GND$1, U$10.GND$2, U$10.GND$3, U$10.GND$4, U$12.2_2, U$13.2, U$13.3, U$20.17, U$20.3, U$20.4, U$20.5, U$20.6, U$20.GND1, U$2G$3.VSS, U$5.GND, U$6.GND, U$8.GND, U$9.GND, U$9.OE; no longer C26.2, JP2.14, JP2.20, JP2.25, JP2.30, JP2.34, JP2.39, JP2.6, JP2.9, JP3.8, R4.2, U$3G$3.VSS, U$4.17, U$4.3, U$4.4, U$4.5, U$4.6, U$4.GND1
- net N$1: now also C17.1, U$1.PXT0, U$3.2; no longer JP2.15
- net N$11: now also IC1.CBUS1, R11.2; no longer JP2.35
- net N$16: now also R1.2, U$6.SEL; no longer JP2.36
- net N$17: now also IC1.!RTS, U$2G$1.NO; no longer JP2.32
- net N$18: now also U$13.1, U$14.A; no longer IC1.CBUS0, R6.2
- net N$2: now also C18.1, U$1.PXT1, U$3.1; no longer R1.2
- net N$5: now also R14.2, U$17.A; no longer IC1.!DTR, U$3G$2.NO
- net N$9: now also IC1.!DTR, U$2G$2.NO; no longer JP2.27
- net P03: now also U$10.A3
- net P04: now also U$9.A7
- net P20: now also U$10.A0
- net P21: now also U$10.A1
- net P22: now also U$10.A2
- net P30: now also U$10.0, U$12.6_1
- net P31: now also U$10.1, U$12.5_1
- net P32: now also U$10.6
- net P33: now also U$10.7
- net P34: now also U$10.A4, U$10.SDA; no longer JP3.5, R9.2
- net P35: now also U$10.A5, U$10.SCL; no longer JP3.6, R10.2
- net P36: now also U$10.13, U$10.SCLK; no longer JP3.4
- net P37: now also U$10.10
- net P42: now also U$10.4
- net P43: now also U$10.5
- net P44: now also U$10.11, U$10.MOSI; no longer JP3.2
- net P45: now also U$10.12, U$10.MISO; no longer JP3.3
- net P50: now also U$10.2; no longer U$7.1, U$7.2
- net P51: now also U$17.C
- net P52: now also U$10.9
- net P53: now also U$10.3; no longer JP3.7
- net P56: now also U$18.C
- net P57: now also U$10.8
- net RESETN: now also U$10.RESETN$1, U$10.RESETN$2, U$7.1, U$7.2
- net RF_CSB: now also U$20.15, U$9.B5; no longer R20.1, R21.1, U$4.15
- net RF_IRQ: now also U$20.13, U$9.B3; no longer JP2.12, U$4.13
- net RF_REGPDIN: now also U$20.10, U$9.B1; no longer JP2.11, U$4.10
- net RF_RSTB: now also U$20.11, U$9.B0; no longer JP2.13, R18.2, U$4.11
- net TEST0: now also U$2G$1.COM; no longer U$3G$1.COM
- net TEST1N: now also U$2G$2.COM; no longer U$3G$2.COM
- net U_TEST0: now also R12.1, U$12.7_1, U$2G$1.NC; no longer R6.1, U$3G$1.NC
- net U_TEST1N: now also R11.1, U$12.4_1, U$2G$2.NC; no longer R5.1, U$3G$2.NC
Other:
- note added: "Naotaka Saito 161229 preriminaly"
- note removed: "(11/MOSI)"
- note removed: "(12/MISO)"
- note removed: "(13/SCK)"
- note removed: "(18/SDA)"
- note removed: "(19/SCL)"
- note removed: "(3/INT1)"
