File: project/PumpMonitoring/PumpMonitoring.sch (EAGLE design)
At the start: 28 parts, among them CN1 NC6-P108-02, Q1 BSS138, Q2 BSS84, Q3 BSS138, Q4 BSS138, Q5 BSS138, T1 IRLML2246, T2 IRLML2246, U1 FSS-71034-10x2,FSS-72034-05x1

Commit message: update pump  monitoring.
Parts:
- removed D8, D9: RRE04EA4D, rohm:RRE04EA4D
- added CN2, CN7: (no value), jst-ph:B5B-PH-K-S
- added CN3, CN6: (no value), jst-ph:B4B-PH-K-S
- added D4, D5: RRE04EA4D, rohm2:RRE04EA4D
- added PAD1, PAD2: (no value), wirepad:1,6/0,9
- added R11, R12: 1K, resistor:R-US_R0603
- added U$1: XB-1-X, lz-shield:XB-1-X
- D1: value VDZ5.1B -> PTZ6.2B; device rohm:VDZXXB -> rohm2:PTZXXB
- D2, D3: device rohm:RRE04EA4D -> rohm2:RRE04EA4D
- R6: value 1k -> 10; device resistor:R-US_R0603 -> rohm2:MCR18
Connections:
- removed net A4: U1D.18
- removed net A5: U1D.19
- removed net VCC5V: C2.+, D2D1.C, D2D2.C, D3D1.C, D3D2.C, U1B.VCC5V_0, U1B.VCC5V_1
- new net +3V3: CN2.2, CN3.2, CN6.2, CN7.2, R11.2, R12.2, U$1.3V3_1, U1B.VCC3V_0, U1B.VCC3V_1
- new net +5V: C2.+, D2D1.C, D2D2.C, D3D1.C, D3D2.C, U$1.5V_1, U1B.VCC5V_0, U1B.VCC5V_1
- new net 0: U$1.0_1, U1B.0
- new net 1: U$1.1_1, U1B.1
- new net N$3: D3D2.A, PAD1.P
- new net SCL: CN2.4, CN6.4, R11.1, U1D.19
- new net SDA: CN2.3, CN6.3, R12.1, U1D.18
- net 5: now also CN2.5
- net A1: now also CN7.4
- net A2: now also CN3.3, CN7.5
- net A3: now also CN3.4
- net GND: now also CN2.1, CN3.1, CN6.1, CN7.1, D4D1.A, D5D2.A, PAD2.P, U$1.GND_1; no longer D8D1.A, D9D1.A
- net I+: now also D4D1.C, D4D2.A; no longer D9D1.C, D9D2.A
- net I-: now also D5D1.A, D5D2.C; no longer D8D1.C, D8D2.A
- net IOUT: now also D4D2.C, D5D1.C; no longer D8D2.C, D9D2.C
- net TEST0: now also U$1.TEST0_1
- net TEST1N: now also U$1.TEST1N_1
Other:
- note added: "A1"
- note added: "I2C"
- note added: "MOTION"
- note added: "SOUND"
- moved on the sheet: C2, D2D2, D3D1, D3D2, V1

Commit message: modify schematic of sound detect module.
Parts:
- removed PAD1, PAD2: (no value), wirepad:1,6/0,9
- added CN4: (no value), jst-ph:B2B-PH-K-S
Connections:
- net GND: now also CN4.2; no longer PAD2.P
- net N$3: now also CN4.1; no longer PAD1.P
Changed lines of the file:
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@@
 <part name="CN1" library="lz-shield" deviceset="TE-NC6-P108-02" device="" value="NC6-P108-02"/>
 <part name="U$2" library="con-hirose" deviceset="MICRO-USB-SHIELD-" device="ZX62R-B-5P" value="ZX62R-B-5P"/>
-<part name="D1" library="rohm2" deviceset="PTZXXB" device="" value="PTZ6.2B"/>
-<part name="V1" library="mouser" deviceset="BAT-HLD-001-THM" device=""/>
 <part name="GND6" library="supply1" deviceset="GND" device=""/>
 <part name="D4" library="rohm2" deviceset="RRE04EA4D" device=""/>
@@
 <part name="+3V1" library="supply1" deviceset="+3V3" device=""/>
 <part name="+3V2" library="supply1" deviceset="+3V3" device=""/>
-<part name="PAD1" library="wirepad" deviceset="1,6/0,9" device=""/>
-<part name="PAD2" library="wirepad" deviceset="1,6/0,9" device=""/>
 <part name="GND12" library="supply1" deviceset="GND" device=""/>
 <part name="U$1" library="lz-shield" deviceset="XB-1-X" device=""/>
@@
 <part name="+3V4" library="supply1" deviceset="+3V3" device=""/>
 <part name="GND14" library="supply1" deviceset="GND" device=""/>
+<part name="CN4" library="jst-ph" deviceset="B2B-PH-*" device="K-S"/>
+<part name="D1" library="rohm2" deviceset="PTZXXB" device="" value="PTZ6.2B"/>
+<part name="V1" library="mouser" deviceset="BAT-HLD-001-THM" device=""/>
 </parts>
 <sheets>
@@
 <instance part="U$2" gate="G$1" x="35.56" y="53.34"/>
 <instance part="U$2" gate="G$2" x="20.32" y="63.5" rot="R180"/>
-<instance part="D1" gate="G$1" x="91.44" y="121.92"/>
-<instance part="V1" gate="G$1" x="218.44" y="88.9"/>
 <instance part="GND6" gate="1" x="218.44" y="78.74"/>
 <instance part="D4" gate="D1" x="81.28" y="132.08" rot="R90"/>
@@
 <instance part="+3V1" gate="G$1" x="302.26" y="157.48"/>
 <instance part="+3V2" gate="G$1" x="373.38" y="187.96"/>
-<instance part="PAD1" gate="1" x="238.76" y="99.06"/>
-<instance part="PAD2" gate="1" x="238.76" y="93.98"/>
 <instance part="GND12" gate="1" x="243.84" y="86.36"/>
 <instance part="U$1" gate="G$1" x="314.96" y="182.88" rot="R180"/>
@@
 <instance part="+3V4" gate="G$1" x="302.26" y="86.36"/>
 <instance part="GND14" gate="1" x="304.8" y="27.94"/>
+<instance part="CN4" gate="G$1" x="248.92" y="99.06"/>
+<instance part="D1" gate="G$1" x="91.44" y="121.92"/>
+<instance part="V1" gate="G$1" x="218.44" y="88.9"/>
 </instances>
 <busses>
@@
 <wire x1="93.98" y1="121.92" x2="104.14" y2="121.92" width="0.1524" layer="91"/>
 <junction x="104.14" y="121.92"/>
-<pinref part="D1" gate="G$1" pin="C"/>
 <pinref part="D4" gate="D2" pin="C"/>
 <pinref part="D5" gate="D1" pin="C"/>
+<pinref part="D1" gate="G$1" pin="C"/>
 </segment>
 </net>
@@
 <wire x1="88.9" y1="121.92" x2="81.28" y2="121.92" width="0.1524" layer="91"/>
 <junction x="81.28" y="121.92"/>
-<pinref part="D1" gate="G$1" pin="A"/>
 <pinref part="D4" gate="D1" pin="A"/>
 <pinref part="D5" gate="D2" pin="A"/>
+<pinref part="D1" gate="G$1" pin="A"/>
 </segment>
 <segment>
@@
 <segment>
 <pinref part="GND6" gate="1" pin="GND"/>
+<wire x1="218.44" y1="81.28" x2="218.44" y2="86.36" width="0.1524" layer="91"/>
 <pinref part="V1" gate="G$1" pin="GND"/>
-<wire x1="218.44" y1="81.28" x2="218.44" y2="86.36" width="0.1524" layer="91"/>
-</segment>
-<segment>
-<pinref part="PAD2" gate="1" pin="P"/>
+</segment>
+<segment>
 <pinref part="GND12" gate="1" pin="GND"/>
-<wire x1="241.3" y1="93.98" x2="243.84" y2="93.98" width="0.1524" layer="91"/>
-<wire x1="243.84" y1="93.98" x2="243.84" y2="88.9" width="0.1524" layer="91"/>
+<wire x1="243.84" y1="96.52" x2="243.84" y2="88.9" width="0.1524" layer="91"/>
+<pinref part="CN4" gate="G$1" pin="2"/>
+<wire x1="248.92" y1="96.52" x2="243.84" y2="96.52" width="0.1524" layer="91"/>
 </segment>
 <segment>
@@
 <net name="N$2" class="0">
 <segment>
-<pinref part="V1" gate="G$1" pin="VDD"/>
 <wire x1="218.44" y1="93.98" x2="218.44" y2="104.14" width="0.1524" layer="91"/>
 <pinref part="D3" gate="D1" pin="A"/>
+<pinref part="V1" gate="G$1" pin="VDD"/>
 </segment>
 </net>
@@
 <net name="N$3" class="0">
 <segment>
-<pinref part="PAD1" gate="1" pin="P"/>
 <pinref part="D3" gate="D2" pin="A"/>
-<wire x1="241.3" y1="99.06" x2="243.84" y2="99.06" width="0.1524" layer="91"/>
 <wire x1="243.84" y1="99.06" x2="243.84" y2="104.14" width="0.1524" layer="91"/>
-</segment>
-</net>
+<pinref part="CN4" gate="G$1" pin="1"/>
+<wire x1="248.92" y1="99.06" x2="243.84" y2="99.06" width="0.1524" layer="91"/>
+</segment>
+</net>
