File: project/PumpMonitoring/MotionSensorModule.sch (EAGLE design)
At the start: 11 parts, among them IC1 LSM9DS1

Commit message: update motion sensor and sound detector modules
Parts:
- removed R3, R4: 10K, resistor:R-US_R0603
- added JMP1, JMP2: 0R-JUMPB, jump-0r-smd:0R-JUMPB
- CN1: value (none) -> JST-PH-K*; device jst-ph:B5B-PH-K-S -> jst-ph:B5B-PH-SM4-TB
Connections:
- removed net N$5: C3.1
- new net N$4: IC1.SDO_A/G, JMP1-0R.2
- new net N$6: IC1.SDO_M, JMP2-0R.2
- net GND: now also CN1.1, JMP1-0R.3, JMP2-0R.3; no longer CN1.2, IC1.SDO_A/G, IC1.SDO_M
- net N$2: now also R2.1; no longer R4.1
- net N$3: now also R1.1; no longer R3.1
- net SCL: now also CN1.4; no longer CN1.3, R1.1
- net SDA: now also CN1.3; no longer CN1.4, R2.1
- net VDD: now also C3.1, CN1.2, JMP1-0R.1, JMP2-0R.1; no longer CN1.1, R3.2, R4.2
Other:
- note added: "I2C Address JMP1(Accel/Gyro) : 0=0x6A (1=0x6B) JMP2(Mag) : 0=0x1C (1=0x1E)"
- note removed: "I2C Address Accel/Gyro : 0x6A Mag : 0x1C"
- moved on the sheet: C1, C2, C3, C4, C5, CN1, IC1, R1, R2

Commit message: add ti.lbr and update motion/sound module
Parts:
- renumbered JMP1 to JP1, JMP2 to JP2
Changed lines of the file:
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@@
 <part name="GND7" library="supply1" deviceset="GND" device=""/>
 <part name="FRAME2" library="frames" deviceset="A4L-LOC" device="" value="MotionSensorModule"/>
-<part name="JMP1" library="jump-0r-smd" deviceset="0R-JUMP" device="B"/>
-<part name="JMP2" library="jump-0r-smd" deviceset="0R-JUMP" device="B"/>
+<part name="JP1" library="jump-0r-smd" deviceset="0R-JUMP" device="B"/>
+<part name="JP2" library="jump-0r-smd" deviceset="0R-JUMP" device="B"/>
 <part name="CN1" library="jst-ph" deviceset="B5B-PH-*" device="SM4-TB" value="JST-PH-K*"/>
+<part name="VDD3" library="supply1" deviceset="VDD" device=""/>
 </parts>
 <sheets>
@@
 <instance part="GND4" gate="1" x="160.02" y="60.96"/>
 <instance part="GND5" gate="1" x="119.38" y="60.96"/>
-<instance part="GND6" gate="1" x="111.76" y="60.96"/>
+<instance part="GND6" gate="1" x="76.2" y="60.96"/>
 <instance part="R1" gate="G$1" x="73.66" y="114.3" rot="R90"/>
 <instance part="R2" gate="G$1" x="66.04" y="114.3" rot="R90"/>
@@
 <instance part="GND7" gate="1" x="58.42" y="60.96"/>
 <instance part="FRAME2" gate="G$1" x="0" y="0"/>
-<instance part="JMP1" gate="-0R" x="58.42" y="132.08" smashed="yes">
+<instance part="JP1" gate="-0R" x="58.42" y="132.08" smashed="yes">
 <attribute name="NAME" x="62.23" y="134.62" size="1.778" layer="95" rot="R90"/>
 </instance>
-<instance part="JMP1" gate="G$2" x="55.88" y="134.62" smashed="yes"/>
-<instance part="JMP2" gate="-0R" x="50.8" y="104.14" smashed="yes">
+<instance part="JP1" gate="G$2" x="55.88" y="134.62" smashed="yes"/>
+<instance part="JP2" gate="-0R" x="50.8" y="104.14" smashed="yes">
 <attribute name="NAME" x="54.61" y="106.68" size="1.778" layer="95" rot="R90"/>
 </instance>
-<instance part="JMP2" gate="G$2" x="48.26" y="106.68"/>
+<instance part="JP2" gate="G$2" x="48.26" y="106.68"/>
 <instance part="CN1" gate="G$1" x="193.04" y="96.52" rot="R180"/>
+<instance part="VDD3" gate="G$1" x="160.02" y="109.22"/>
 </instances>
 <busses>
@@
 <wire x1="111.76" y1="86.36" x2="111.76" y2="83.82" width="0.1524" layer="91"/>
 <wire x1="111.76" y1="83.82" x2="111.76" y2="66.04" width="0.1524" layer="91"/>
-<wire x1="111.76" y1="66.04" x2="111.76" y2="63.5" width="0.1524" layer="91"/>
 <wire x1="106.68" y1="86.36" x2="111.76" y2="86.36" width="0.1524" layer="91"/>
 <pinref part="IC1" gate="G$1" pin="RES5"/>
@@
 <pinref part="IC1" gate="G$1" pin="RES4"/>
 <wire x1="96.52" y1="68.58" x2="96.52" y2="66.04" width="0.1524" layer="91"/>
-<junction x="111.76" y="66.04"/>
 <junction x="111.76" y="83.82"/>
 <junction x="111.76" y="86.36"/>
@@
 <junction x="93.98" y="66.04"/>
 <junction x="88.9" y="66.04"/>
+<wire x1="86.36" y1="66.04" x2="76.2" y2="66.04" width="0.1524" layer="91"/>
+<wire x1="76.2" y1="66.04" x2="76.2" y2="63.5" width="0.1524" layer="91"/>
+<junction x="86.36" y="66.04"/>
 </segment>
 <segment>
@@
 </segment>
 <segment>
-<pinref part="JMP1" gate="-0R" pin="3"/>
+<pinref part="JP1" gate="-0R" pin="3"/>
 <pinref part="GND7" gate="1" pin="GND"/>
 <wire x1="58.42" y1="129.54" x2="58.42" y2="91.44" width="0.1524" layer="91"/>
-<pinref part="JMP2" gate="-0R" pin="3"/>
+<pinref part="JP2" gate="-0R" pin="3"/>
 <wire x1="58.42" y1="91.44" x2="58.42" y2="63.5" width="0.1524" layer="91"/>
 <wire x1="50.8" y1="101.6" x2="50.8" y2="91.44" width="0.1524" layer="91"/>
@@
 <net name="VDD" class="0">
 <segment>
-<pinref part="IC1" gate="G$1" pin="VDD1"/>
-<wire x1="106.68" y1="96.52" x2="149.86" y2="96.52" width="0.1524" layer="91"/>
-<wire x1="149.86" y1="96.52" x2="149.86" y2="99.06" width="0.1524" layer="91"/>
-<pinref part="IC1" gate="G$1" pin="VDD2"/>
-<wire x1="149.86" y1="99.06" x2="149.86" y2="127" width="0.1524" layer="91"/>
-<wire x1="106.68" y1="99.06" x2="149.86" y2="99.06" width="0.1524" layer="91"/>
-<junction x="149.86" y="99.06"/>
-<pinref part="C4" gate="G$1" pin="1"/>
-<wire x1="160.02" y1="76.2" x2="160.02" y2="83.82" width="0.1524" layer="91"/>
-<wire x1="160.02" y1="83.82" x2="160.02" y2="127" width="0.1524" layer="91"/>
-<wire x1="160.02" y1="127" x2="149.86" y2="127" width="0.1524" layer="91"/>
-<junction x="149.86" y="127"/>
 <pinref part="IC1" gate="G$1" pin="VDDIO2"/>
 <wire x1="93.98" y1="124.46" x2="93.98" y2="127" width="0.1524" layer="91"/>
@@
 <junction x="139.7" y="104.14"/>
 <wire x1="139.7" y1="127" x2="139.7" y2="104.14" width="0.1524" layer="91"/>
-<wire x1="139.7" y1="127" x2="149.86" y2="127" width="0.1524" layer="91"/>
 <junction x="139.7" y="127"/>
 <pinref part="VDD1" gate="G$1" pin="VDD"/>
 <wire x1="139.7" y1="137.16" x2="139.7" y2="127" width="0.1524" layer="91"/>
-<pinref part="C3" gate="G$1" pin="1"/>
-<wire x1="149.86" y1="76.2" x2="149.86" y2="83.82" width="0.1524" layer="91"/>
-<wire x1="149.86" y1="83.82" x2="160.02" y2="83.82" width="0.1524" layer="91"/>
-<junction x="160.02" y="83.82"/>
 </segment>
 <segment>
@@
 <wire x1="66.04" y1="119.38" x2="66.04" y2="124.46" width="0.1524" layer="91"/>
 <wire x1="66.04" y1="124.46" x2="73.66" y2="124.46" width="0.1524" layer="91"/>
-<pinref part="JMP1" gate="-0R" pin="1"/>
+<pinref part="JP1" gate="-0R" pin="1"/>
 <wire x1="58.42" y1="134.62" x2="58.42" y2="147.32" width="0.1524" layer="91"/>
 <wire x1="58.42" y1="147.32" x2="73.66" y2="147.32" width="0.1524" layer="91"/>
 <junction x="73.66" y="147.32"/>
-<pinref part="JMP2" gate="-0R" pin="1"/>
+<pinref part="JP2" gate="-0R" pin="1"/>
 <wire x1="50.8" y1="106.68" x2="50.8" y2="147.32" width="0.1524" layer="91"/>
 <wire x1="50.8" y1="147.32" x2="58.42" y2="147.32" width="0.1524" layer="91"/>
@@
 <label x="205.74" y="93.98" size="1.778" layer="95"/>
 <pinref part="CN1" gate="G$1" pin="2"/>
+</segment>
+<segment>
+<pinref part="IC1" gate="G$1" pin="VDD2"/>
+<wire x1="106.68" y1="99.06" x2="111.76" y2="99.06" width="0.1524" layer="91"/>
+<pinref part="IC1" gate="G$1" pin="VDD1"/>
+<wire x1="106.68" y1="96.52" x2="111.76" y2="96.52" width="0.1524" layer="91"/>
+<pinref part="C4" gate="G$1" pin="1"/>
+<wire x1="111.76" y1="96.52" x2="160.02" y2="96.52" width="0.1524" layer="91"/>
+<wire x1="160.02" y1="76.2" x2="160.02" y2="91.44" width="0.1524" layer="91"/>
+<pinref part="C3" gate="G$1" pin="1"/>
+<wire x1="160.02" y1="96.52" x2="160.02" y2="91.44" width="0.1524" layer="91"/>
+<junction x="160.02" y="96.52"/>
+<junction x="160.02" y="91.44"/>
+<pinref part="VDD3" gate="G$1" pin="VDD"/>
+<wire x1="160.02" y1="106.68" x2="160.02" y2="96.52" width="0.1524" layer="91"/>
+<wire x1="111.76" y1="99.06" x2="111.76" y2="96.52" width="0.1524" layer="91"/>
+<junction x="111.76" y="96.52"/>
+<wire x1="149.86" y1="76.2" x2="149.86" y2="91.44" width="0.1524" layer="91"/>
+<wire x1="149.86" y1="91.44" x2="160.02" y2="91.44" width="0.1524" layer="91"/>
 </segment>
 </net>
@@
 <segment>
 <pinref part="IC1" gate="G$1" pin="SDO_A/G"/>
-<pinref part="JMP1" gate="-0R" pin="2"/>
+<pinref part="JP1" gate="-0R" pin="2"/>
 <wire x1="60.96" y1="132.08" x2="86.36" y2="132.08" width="0.1524" layer="91"/>
 <wire x1="86.36" y1="132.08" x2="86.36" y2="124.46" width="0.1524" layer="91"/>
@@
 <net name="N$6" class="0">
 <segment>
-<pinref part="JMP2" gate="-0R" pin="2"/>
+<pinref part="JP2" gate="-0R" pin="2"/>
 <pinref part="IC1" gate="G$1" pin="SDO_M"/>
 <wire x1="53.34" y1="104.14" x2="78.74" y2="104.14" width="0.1524" layer="91"/>
