File: project/PumpMonitoring/SoundDetectorModule.brd (EAGLE design)
At the start: 46 x 22 mm, 32 parts, among them CN1 JST-PH-K*, IC1 LMV324

Commit message: update sound detector(added license information)
Other:
- board text added: "This document is released under Creative Commons ShareAlike4.0 International license. Original URL: https://github.com/sparkfun/Sound_Detector"
Changed lines of the file:
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@@
 <layer number="49" name="Reference" color="7" fill="1" visible="no" active="yes"/>
 <layer number="50" name="dxf" color="7" fill="1" visible="no" active="no"/>
-<layer number="51" name="tDocu" color="7" fill="1" visible="no" active="yes"/>
+<layer number="51" name="tDocu" color="7" fill="1" visible="yes" active="yes"/>
 <layer number="52" name="bDocu" color="7" fill="1" visible="no" active="yes"/>
 <layer number="53" name="tGND_GNDA" color="7" fill="9" visible="no" active="no"/>
@@
 <circle x="5.588" y="10.16" radius="4.819309375" width="0.4064" layer="21"/>
 <wire x1="3.302" y1="13.1826" x2="4.318" y2="13.1826" width="0.254" layer="21"/>
+<text x="-5.588" y="-5.08" size="0.8128" layer="51" font="fixed">This document is released under Creative Commons ShareAlike4.0 International license.
+Original URL: https://github.com/sparkfun/Sound_Detector </text>
 </plain>
 <attributes>
@@
 </board>
 </drawing>
+<compatibility>
+<note version="6.3" minversion="6.2.2" severity="warning">
+Since Version 6.2.2 text objects can contain more than one line,
+which will not be processed correctly with this version.
+</note>
+</compatibility>
 </eagle>
