File: project/PumpMonitoring/171020_PumpMonitoring/eagle/PumpMonitoring.brd (EAGLE design)
At the start: 85 x 56 mm, 46 parts, among them CN1 B6B-EH-, CON1 B2B-EH-, CON2 MJ-3536N, CON3 NC6-P108-02, Q1 BSS138, Q2 BSS84, Q3 BSS138, Q4 BSS138, Q5 BSS138, U1 FSS-71034-10x2,FSS-72034-05x1

Commit message: bug fix of pump monitoring.
Parts:
- C3: device rcl:C0603 -> resistor:C0603
Changed lines of the file:
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@@
 </element>
 <element name="CN1" library="jst-ph" package="B6B-EH" value="B6B-EH-" x="44.45" y="11.43" rot="MR90"/>
-<element name="C3" library="rcl" package="C0603" value="" x="43.18" y="26.67" smashed="yes" rot="R270">
+<element name="C3" library="resistor" package="C0603" value="" x="43.18" y="26.67" smashed="yes" rot="R270">
 <attribute name="NAME" x="44.45" y="27.94" size="1.27" layer="25" rot="R270"/>
 <attribute name="VALUE" x="41.275" y="27.305" size="1.27" layer="27" rot="R270"/>
