File: project/PumpMonitoring/171020_PumpMonitoring/eagle/PumpMonitoring.sch (EAGLE design)
At the start: 45 parts, among them CN1 B6B-EH-, CON1 B2B-EH-, CON2 MJ-3536N, CON3 NC6-P108-02, Q1 BSS138, Q2 BSS84, Q3 BSS138, Q4 BSS138, Q5 BSS138, U1 FSS-71034-10x2,FSS-72034-05x1

Commit message: bug fix of pump monitoring.
Parts:
- C3: device rcl:C-USC0603 -> resistor:C-USC0603
Changed lines of the file:
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@@
 <part name="CN1" library="jst-ph" deviceset="B6B-EH-*" device=""/>
 <part name="FRAME1" library="frames" deviceset="A3L-LOC" device=""/>
-<part name="C3" library="rcl" deviceset="C-US" device="C0603"/>
+<part name="C3" library="resistor" deviceset="C-US" device="C0603"/>
 </parts>
 <sheets>
